Commit message: real mapping

File: src/ep_driver/urdf/ep_description.xacro (robot description, xacro)
@@ -12,10 +12,10 @@
     <parent link="base_link"/>
     <child link="laser_link"/>
-    <origin rpy="0 0 3.1415926535897" xyz="0.12 0 0.1"/>
+    <origin rpy="0 0 3.1415926535897" xyz="0.12 0 0.07"/>
   </joint>
   <joint name="base_to_imu_joint" type="fixed">
     <parent link="base_link"/>
     <child link="imu_link"/>
-    <origin rpy="0 0 0" xyz="0 0 0.08"/>
+    <origin rpy="0 0 0" xyz="0 0 0"/>
   </joint>
   <joint name="base_to_arm_joint" type="fixed">
